File: evnotipi-hat.sch (KiCad schematic (older format))
At the start: 2 parts, among them J1 RPi_GPIO, J2 RPi_GPIO

Commit message: Redesigned again. Prototype 1
Parts:
- removed J2: RPi_GPIO, RPi_Hat:Pin_Header_Straight_2x20, symbol Connector-ML:RPi_GPIO
- added C1, C2: 10µF, Capacitor_SMD:C_0805_2012Metric_Pad1.15x1.40mm_HandSolder, symbol Device:C
- added C3, C4: 100nF, Capacitor_SMD:C_0805_2012Metric_Pad1.15x1.40mm_HandSolder, symbol Device:C
- added C5, C6: 22µF, Capacitor_SMD:C_0805_2012Metric_Pad1.15x1.40mm_HandSolder, symbol Device:C
- added D1: D_Schottky, Diode_SMD:D_SOD-128, symbol Device:D_Schottky
- added D9: blue, LED_SMD:LED_0603_1608Metric, symbol Device:LED
- added J2: DB9_Male_MountingHoles, Connector_Dsub:DSUB-9_Male_Horizontal_P2.77x2.84mm_EdgePinOffset4.94mm_Housed_MountingHolesOffset7.48mm, symbol Connector:DB9_Male_MountingHoles
- added L1: 5,6µH, Inductor_SMD:L_Coilcraft_XAL60xx_6.36x6.56mm, symbol Device:L
- added R1: R10k, Resistor_SMD:R_0603_1608Metric_Pad1.05x0.95mm_HandSolder, symbol Device:R
- added R18: R15, Resistor_SMD:R_0603_1608Metric_Pad1.05x0.95mm_HandSolder, symbol Device:R
- added R19: 10K, Resistor_SMD:R_0603_1608Metric_Pad1.05x0.95mm_HandSolder, symbol Device:R
- added R2: 30R, Resistor_SMD:R_0603_1608Metric_Pad1.05x0.95mm_HandSolder, symbol Device:R
- added R3: 52,3k, Resistor_SMD:R_0603_1608Metric_Pad1.05x0.95mm_HandSolder, symbol Device:R
- added SW2: SW_Reset, Button_Switch_SMD:SW_SPST_B3U-1000P, symbol Switch:SW_Push
- added U1: TPS56339DDC, Package_TO_SOT_SMD:SOT-23-6, symbol Regulator_Switching:TPS56339DDC
- J1: footprint RPi_Hat:Samtec_HLE-120-02-XXX-DV-BE-XX-XX -> Connector_Samtec_HLE_SMD-ML:Samtec_HLE-120-02-xxx-DV-BE-A_2x20_RPi_Top
Connections:
- net +3V3: now reaches J1.1 (3.3V)
- net +3V3: now also J1.17 (3.3V)
- net RPI_LED: now reaches J1.11 (GPIO17)
- net RPI_LED: now also R18.2
- net RPI_CMD: now reaches J1.13 (GPIO27)
- net RPI_CMD: now also SW2.1
- net GND: now reaches J1.14 (GND)
- net GND: now also J1.20 (GND), J1.25 (GND), J1.30 (GND), J1.34 (GND), J1.39 (GND), J1.6 (GND), J1.9 (GND), C1.2, C2.2, C3.2, C5.2, C6.2, D9.1 (K), J2.1, J2.2, R1.2, R19.1, U1.1 (GND)
- net MOSI: now reaches J1.19 (GPIO10_SPI_MOSI)
- net +5V: now reaches J1.2 (5V)
- net +5V: now also J1.4 (5V), C5.1, C6.1, L1.1, R3.1
- net MISO: now reaches J1.21 (GPIO09_SPI_MISO)
- net RXINT: now reaches J1.22 (GPIO25)
- net SPI_CLK: now reaches J1.23 (GPIO11_SPI_CLK)
- net SPI_CE0: now reaches J1.24 (GPIO08_SPI_CE0_N)
- net SDA: now reaches J1.3 (GPIO02_SDA1_I2C)
- net PCIE_PWR_EN: now reaches J1.35 (GPIO19)
- net Pi_Running: now reaches J1.37 (GPIO26)
- net SCL: now reaches J1.5 (GPIO03_SCL1_I2C)
- new net: C4.1, L1.2, U1.2 (SW)
- new net: C4.2, R2.1
- new net: R1.1, R3.2, U1.4 (FB)
- new net: R2.2, U1.6 (BOOT)
- new net: D9.2 (A), R18.1
- new net: R19.2, SW2.2
- new net +12P: D1.2 (A), J2.9
- new net +12V: C1.1, C2.1, C3.1, D1.1 (K), U1.3 (VIN)
- new net CAN_H: J2.6
- new net CAN_L: J2.5
- new net PWR_EN: U1.5 (EN)
- no-connect marks 0 -> 17
Other:
- note added: "12V to 5V 3A DC-DC"
- note added: "Button and assiciated status LED. Might be used for factory reset or reboot."
- note removed: "Socket on bottom"
- note removed: "Surface Mount Connector"
- note removed: "Thru-Hole Connector"
- moved on the sheet: J1
